File: G_FY2015_Mez.sch (EAGLE design)
At the start: 99 parts, among them IC100 FT232RL, J1 RPI2_GPIO_HOLES, J100 TOKUDEN_SP6, J300 SHV_PIGTAIL_LAND, J301 SHV_PIGTAIL_LAND, U1 AD8138, U10 LM60, U100 AD9215, U101 AD8138, U11 MCP4822-E/SN, U110 AD9215, U120 AD9215, U130 AD9215, U2 AD8138, U3 AD8138, U300 OPTON_1PA_12, U301 OPTON_1PA_12, U4 LT6106, U5 MCP3208-CI/SL, U6 MCP1525TSOT-23-3, U7 LM60, U8 LM60, U9 LM60

Commit message: G_FY2015_Mez.sch - completed first drafting
Parts:
- removed JP_SLOWADC: (no value), pinhead:PINHD-2X4
- added C100, C110, C120, C130: 100p, Aardvark:C226-3216
- added C101, C111, C121, C131: ???, Aardvark:C226-3216
- added C102, C103, C112, C113, C122, C123, C132, C133: 0.1u, Aardvark:C226-3216
- added C190, C192: 100n, Aardvark:C226-3216
- added C191, C193: 4.7u, Aardvark:C226-3216
- added C194: 0.01u, Aardvark:C226-3216
- added C195, C601, C611, C620, C621: 10u, Aardvark:C226-3216
- added C600, C610: 100u, rcl:CPOL-USE2.5-5
- added C622: 1u, Aardvark:C226-3216
- added J102, J103: EPL.00.250.NTN, Aardvark:EPL.00.250.NTN
- added J180: TOKUDEN_SP6, Aardvark:TOKUDEN_SP6
- added J181: (no value), Aardvark:MINI-USB-RCPT-B-5PS-R/A-SMD(ST-USB-002A)
- added J600_12V: IL-4P-S3EN2, Aardvark:IL-4P-S3EN2
- added J610: 2.1MMJACKTHM, Aardvark:2.1MMJACKTHM
- added JP2: (no value), pinhead:PINHD-2X2
- added R107, R117, R127, R137: 1M, Aardvark:R2012
- added R108, R118, R128, R138: ???, Aardvark:R2012
- added R197, R198, R199: 330, Aardvark:R2012
- added R302, R511: 100, Aardvark:R2012
- added R303: 4.7k, Aardvark:R2012
- added R510: 0.1, Aardvark:R_LVR03
- added R512: 10k, Aardvark:R2012
- added R600: 280, Aardvark:R2012
- added R610: 2k, Aardvark:R2012
- added TP100, TP101, TP102, TP104, TP_1PPS, TP_PRE_IN1, TP_PRE_IN2, TP_PRE_IN3, TP_PRE_IN4, TP_PRE_OUT0, TP_PRE_OUT1, TP_PRE_OUT2, TP_PRE_OUT3: TPPAD1-17, Aardvark:TPPAD1-17
- added U$17, U$18, U$19, U$20, U$21: NC, Aardvark:NC
- added U$23: 2SJ313, Aardvark:2SJ313
- added U102, U112, U122, U132: (no value), Aardvark:LM6172SOIC(D)8
- added U191: GPS_FGPMMOPA6H, Aardvark:GPS_FGPMMOPA6H
- added U192: LED-5, Aardvark:LED-5
- added U302: 2SC1815, Aardvark:2SC1815
- added U510: LT6106, Aardvark:LT6106
- added U600, U610: PHT12050WAH, Aardvark:PHT12050WAH
- added U620: LTC1983ES6-3, Aardvark:LTC1983ES6-3
- added VR100, VR110, VR120, VR130, VR300, VR301: (no value), Aardvark:DIP-TRIMMER-10K-10%-1/2W(3P-9.7X5.0X9.80MM)
- J100: value TOKUDEN_SP6 -> EPL.00.250.NTN; device Aardvark:TOKUDEN_SP6 -> Aardvark:EPL.00.250.NTN
- J101: value (none) -> EPL.00.250.NTN; device Aardvark:MINI-USB-RCPT-B-5PS-R/A-SMD(ST-USB-002A) -> Aardvark:EPL.00.250.NTN
- R300, R301: value (none) -> 47k; device Aardvark:DIP-TRIMMER-10K-10%-1/2W(3P-9.7X5.0X9.80MM) -> Aardvark:R2012
- renumbered R2 to R500, R3 to R501, R4 to R502, TP1 to TP103, TP2 to TP113, TP3 to TP123, TP4 to TP133, U$13 to U190, U4 to U500
Connections:
- removed net FPGA_RX: J1.GPIO14, J100.B_24
- removed net FPGA_TX: J1.GPIO15, J100.B_22
- removed net UART_DTS: J100.A_2
- removed net UART_RX: IC100.TXD, J100.A_1
- removed net UART_TX: IC100.RXD, J100.A_0
- new net +3V3_BEFORE_SENSE: R510.P$2, R511.1, U510PWR.V+
- new net +5V_BEFORE_SENSE: R500.P$2, R501.1, U500PWR.V+
- new net 3V3_BEFORE_SENSE: U610.V_O
- new net 5V_BEFORE_SENSE: U600.V_O
- new net BBB: J180.A_2
- new net FT232_RX_FPGA_TX: IC100.RXD, J180.A_0
- new net FT232_TX_FPGA_RX: IC100.TXD, J180.A_1
- new net HV_PWR_12V: U$23.D, U300.VIN, U301.VIN
- new net HV_PWR_ENADIS: J1.GPIO16, R302.2
- new net N$54: C100.2, C101.1, R107.1, U102A.OUT
- new net N$55: C101.2, R108.1, U102B.+
- new net N$58: C100.1, J100.1, R107.2, TP_PRE_IN1.TP, U102A.-
- new net N$59: U$17.NC, U600.INHIBIT
- new net N$60: R197.1, U191.TX
- new net N$61: C110.2, C111.1, R117.1, U112A.OUT
- new net N$62: U102B.-, VR100.2
- new net N$63: C111.2, R118.1, U112B.+
- new net N$64: U$18.NC, U191.VBACKUP
- new net N$65: R199.2, U191.3D_FIX
- new net N$66: U$20.NC, U191.EX_ANT
- new net N$67: U$21.NC, U191.RTCM
- new net N$68: R198.1, U191.RX
- new net N$69: R199.1, U192.A
- new net N$70: C110.1, J101.1, R117.2, TP_PRE_IN2.TP, U112A.-
- new net N$71: R610.2, U610.ADJUST
- new net N$72: U112B.-, VR110.2
- new net N$73: C120.2, C121.1, R127.1, U122A.OUT
- new net N$74: C121.2, R128.1, U122B.+
- new net N$75: C120.1, J102.1, R127.2, TP_PRE_IN3.TP, U122A.-
- new net N$76: U$19.NC, U610.INHIBIT
- new net N$77: U122B.-, VR120.2
- new net N$78: C130.2, C131.1, R137.1, U132A.OUT
- new net N$79: C131.2, R138.1, U132B.+
- new net N$80: C130.1, J103.1, R137.2, TP_PRE_IN4.TP, U132A.-
- new net N$81: C622.2, U620.C+
- new net N$82: U132B.-, VR130.2
- new net N$83: C622.1, U620.C-
- new net N$84: R600.2, U600.ADJUST
- new net N$85: R300.1, R301.2, U$23.G
- new net N$86: R301.1, U302.C
- new net N$87: R302.1, R303.1, U302.B
- new net PREAMP0_OUT: TP_PRE_OUT0.TP, U102B.OUT, VR100.3
- new net PREAMP1_OUT: TP_PRE_OUT1.TP, U112B.OUT, VR110.3
- new net PREAMP2_OUT: TP_PRE_OUT2.TP, U122B.OUT, VR120.3
- new net PREAMP3_OUT: TP_PRE_OUT3.TP, U132B.OUT, VR130.3
- new net RPI_RX_FPGA_TX: J1.GPIO15, J180.B_22
- new net RPI_TX_FPGA_RX: J1.GPIO14, J180.B_24
- net +12V: now also C600.+, C601.2, C610.+, C611.2, J600_12V.1, J600_12V.2, J610.TIP, R300.2, U$23.S, U600.TRACK, U600.V_I, U610.TRACK, U610.V_I; no longer U300.VIN, U301.VIN
- net +3V3: now also C102.2, C112.2, C122.2, C132.2, C190.1, C191.1, C192.2, C193.2, C194.2, C195.2, R510.P$1, U102P.V+, U112P.V+, U122P.V+, U132P.V+, U191.NRESET, U191.VCC, U510A.+
- net +5V: now also C620.2, J180.V5, U620./SHDN, U620.VCC; no longer J100.V5, R500.P$2, R501.1, U500PWR.V+
- net -3V3: now also C103.2, C113.2, C123.2, C133.2, C621.1, U102P.V-, U112P.V-, U122P.V-, U132P.V-, U620.VOUT
- net AAA: now also J180.B_31; no longer J100.B_31
- net ADC0_CLK: now also J180.B_23, TP104.TP; no longer J100.B_23
- net ADC0_D0: now also J180.B_0; no longer J100.B_0
- net ADC0_D1: now also J180.B_1; no longer J100.B_1
- net ADC0_D2: now also J180.B_2; no longer J100.B_2
- net ADC0_D3: now also J180.B_3; no longer J100.B_3
- net ADC0_D4: now also J180.B_4; no longer J100.B_4
- net ADC0_D5: now also J180.B_5; no longer J100.B_5
- net ADC0_D6: now also J180.B_6; no longer J100.B_6
- net ADC0_D7: now also J180.B_7; no longer J100.B_7
- net ADC0_D8: now also J180.B_8; no longer J100.B_8
- net ADC0_D9: now also J180.B_9; no longer J100.B_9
- net ADC0_VIN_N: now also TP102.TP
- net ADC0_VIN_P: now also TP101.TP
- net ADC1_CLK: now also J180.B_25; no longer J100.B_25
- net ADC1_D0: now also J180.B_10; no longer J100.B_10
- net ADC1_D1: now also J180.B_11; no longer J100.B_11
- net ADC1_D2: now also J180.B_12; no longer J100.B_12
- net ADC1_D3: now also J180.B_13; no longer J100.B_13
- net ADC1_D4: now also J180.B_14; no longer J100.B_14
- net ADC1_D5: now also J180.B_15; no longer J100.B_15
- net ADC1_D6: now also J180.B_16; no longer J100.B_16
- net ADC1_D7: now also J180.B_17; no longer J100.B_17
- net ADC1_D8: now also J180.B_18; no longer J100.B_18
- net ADC1_D9: now also J180.B_19; no longer J100.B_19
- net ADC2_CLK: now also J180.B_27; no longer J100.B_27
- net ADC2_D0: now also J180.A_8; no longer J100.A_8
- net ADC2_D1: now also J180.A_9; no longer J100.A_9
- net ADC2_D2: now also J180.A_10; no longer J100.A_10
- net ADC2_D3: now also J180.A_11; no longer J100.A_11
- net ADC2_D4: now also J180.A_12; no longer J100.A_12
- net ADC2_D5: now also J180.A_13; no longer J100.A_13
- net ADC2_D6: now also J180.A_14; no longer J100.A_14
- net ADC2_D8: now also J180.A_16; no longer J100.A_16
- net ADC2_D9: now also J180.A_17; no longer J100.A_17
- net ADC3_CLK: now also J180.B_29; no longer J100.B_29
- net ADC3_D0: now also J180.A_18; no longer J100.A_18
- net ADC3_D1: now also J180.A_19; no longer J100.A_19
- net ADC3_D2: now also J180.A_20; no longer J100.A_20
- net ADC3_D3: now also J180.A_21; no longer J100.A_21
- net ADC3_D4: now also J180.A_22; no longer J100.A_22
- net ADC3_D5: now also J180.A_23; no longer J100.A_23
- net ADC3_D6: now also J180.A_24; no longer J100.A_24
- net ADC3_D7: now also J180.A_25; no longer J100.A_25
- net ADC3_D8: now also J180.A_26; no longer J100.A_26
- net ADC3_D9: now also J180.A_27; no longer J100.A_27
- net ADC_MODE: now also J180.B_21; no longer J100.B_21
- net ADC_PDWN: now also J180.B_20; no longer J100.B_20
- net AGND: now also C102.1, C103.1, C112.1, C113.1, C122.1, C123.1, C132.1, C133.1, J100.GND, J101.GND, J102.GND, J103.GND, JP2.2, JP2.4, R108.2, R118.2, R128.2, R138.2, U102A.+, U112A.+, U122A.+, U132A.+, VR100.1, VR110.1, VR120.1, VR130.1; no longer JP_SLOWADC.2, JP_SLOWADC.4, JP_SLOWADC.6, JP_SLOWADC.8
- net DIFFAMP0_IN: now also TP100.TP
- net GND: now also C190.2, C191.2, C192.1, C193.1, C194.1, C195.1, C600.-, C601.1, C610.-, C611.1, C620.1, C621.2, J180.GND, J180.GND_3, J180.GND_4, J180.GND_5, J180.GND_6, J180.GND_7, J181.GND@5, J600_12V.3, J600_12V.4, J610.RING, R303.2, R512.1, R600.1, R610.1, U191.GND@12, U191.GND@19, U191.GND@3, U191.GND@8, U192.K, U302.E, U510PWR.V-, U600.GND, U610.GND, U620.GND, VR300.1, VR301.1; no longer J100.GND, J100.GND_3, J100.GND_4, J100.GND_5, J100.GND_6, J100.GND_7, J101.GND@5, R300.2, R301.2
- net GPS_1PPS: now also J180.B_33, TP_1PPS.TP, U191.1PPS; no longer J100.B_33
- net GPS_RX_FPGA_TX: now also J180.B_35, R198.2; no longer J100.B_35
- net GPS_TX_FPGA_RX: now also J180.B_34, R197.2; no longer J100.B_34
- net N$24: now also J180.A_4; no longer J100.A_4
- net N$26: now also J180.A_7; no longer J100.A_7
- net N$27: now also J180.A_5; no longer J100.A_5
- net N$28: now also J180.A_3; no longer J100.A_3
- net N$3: now also VR300.2; no longer R300.3
- net N$34: now also J181.GND@1, J181.GND@2, J181.GND@3, J181.GND@4; no longer J101.GND@1, J101.GND@2, J101.GND@3, J101.GND@4
- net N$5: now also VR300.3; no longer R300.1
- net N$53: now also J180.V33_1, J180.V33_2, J180.V33_3, J180.V33_4; no longer J100.V33_1, J100.V33_2, J100.V33_3, J100.V33_4
- net N$6: now also VR301.2; no longer R301.3
- net N$7: now also VR301.3; no longer R301.1
- net N$9: now also R511.2, U510A.-; no longer R502.2, U500A.OUT
- net NNN: now also J180.A_6; no longer J100.A_6
- net SLOWADC_4: now also R502.2, U500A.OUT; no longer JP_SLOWADC.1
- net SLOWADC_5: now also R512.2, U510A.OUT; no longer JP_SLOWADC.3
- net SLOWADC_6: now also JP2.1; no longer JP_SLOWADC.5
- net SLOWADC_7: now also JP2.3; no longer JP_SLOWADC.7
- net SPW_DIN: now also J180.B_30; no longer J100.B_30
- net SPW_DOUT: now also J180.B_26; no longer J100.B_26
- net SPW_SIN: now also J180.B_32; no longer J100.B_32
- net SPW_SOUT: now also J180.B_28; no longer J100.B_28
- net USB_D_M: now also J181.DM; no longer J101.DM
- net USB_D_P: now also J181.DP; no longer J101.DP
Other:
- note added: "ADC"
- note added: "Current Sense Amp"
- note added: "DCDC +12V=>+3.3V"
- note added: "DCDC +12V=>+5V"
- note added: "DCDC +5V=>-3V"
- note added: "DCDC Modules"
- note added: "FPGA"
- note added: "GPS Module"
- note added: "HV 12V Power Control (from Raspberry Pi)"
- note added: "HVPS Modules"
- note added: "Power Connectors"
- note added: "Pre Amplifier for PMT"
- note added: "Single-end-to-differential Amp"
- note added: "SpaceWire LVDS Tx/Rx"
- note added: "USB-UART"
- note removed: "TODO: Add PMT Amp"
- note removed: "TODO: GPS Module"

Commit message: G_FY2015_Mez.brd - partially placed
Parts:
- added J2: SPACEWIRE_MDMMDM9, Aardvark:SPACEWIRE_MDMMDM9
- renumbered U$23 to U303
Connections:
- new net N$93: J2.GND1
- net GND: now also J2.GND, J2.GND2
- net SPW_DIN_N: now also J2.DIN-
- net SPW_DIN_P: now also J2.DIN+
- net SPW_DOUT_N: now also J2.DOUT-
- net SPW_DOUT_P: now also J2.DOUT+
- net SPW_SIN_N: now also J2.SIN-
- net SPW_SIN_P: now also J2.SIN+
- net SPW_SOUT_N: now also J2.SOUT-
- net SPW_SOUT_P: now also J2.SOUT+
Changed lines of the file:
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@@
 <part name="R302" library="Aardvark" deviceset="R2012" device="" value="100"/>
 <part name="R303" library="Aardvark" deviceset="R2012" device="" value="4.7k"/>
-<part name="U$23" library="Aardvark" deviceset="2SJ313" device=""/>
+<part name="U303" library="Aardvark" deviceset="2SJ313" device=""/>
 <part name="P+5" library="Aardvark" deviceset="+12V" device=""/>
 <part name="P+13" library="Aardvark" deviceset="+5V" device=""/>
+<part name="J2" library="Aardvark" deviceset="SPACEWIRE_MDM" device="MDM9"/>
+<part name="GND55" library="Aardvark" deviceset="GND" device=""/>
 </parts>
 <sheets>
@@
 <instance part="TP_PRE_IN3" gate="G$1" x="-246.38" y="-22.86" rot="R180"/>
 <instance part="TP104" gate="G$1" x="-55.88" y="86.36" rot="R90"/>
+<instance part="J2" gate="G$1" x="292.1" y="116.84"/>
+<instance part="GND55" gate="1" x="271.78" y="119.38" rot="R270"/>
 </instances>
 <busses>
@@
 <pinref part="GND46" gate="1" pin="GND"/>
 </segment>
+<segment>
+<pinref part="J2" gate="G$1" pin="GND2"/>
+<wire x1="287.02" y1="114.3" x2="284.48" y2="114.3" width="0.1524" layer="91"/>
+<pinref part="J2" gate="G$1" pin="GND"/>
+<wire x1="287.02" y1="119.38" x2="284.48" y2="119.38" width="0.1524" layer="91"/>
+<wire x1="284.48" y1="114.3" x2="284.48" y2="119.38" width="0.1524" layer="91"/>
+<wire x1="284.48" y1="119.38" x2="274.32" y2="119.38" width="0.1524" layer="91"/>
+<pinref part="GND55" gate="1" pin="GND"/>
+</segment>
 </net>
 <net name="N$10" class="0">
@@
 <junction x="241.3" y="144.78"/>
 </segment>
+<segment>
+<pinref part="J2" gate="G$1" pin="DIN-"/>
+<wire x1="287.02" y1="132.08" x2="284.48" y2="132.08" width="0.1524" layer="91"/>
+<label x="269.24" y="132.08" size="1.778" layer="95"/>
+</segment>
 </net>
 <net name="SPW_DIN_P" class="0">
@@
 <junction x="241.3" y="134.62"/>
 </segment>
+<segment>
+<pinref part="J2" gate="G$1" pin="DIN+"/>
+<wire x1="287.02" y1="134.62" x2="284.48" y2="134.62" width="0.1524" layer="91"/>
+<label x="269.24" y="134.62" size="1.778" layer="95"/>
+</segment>
 </net>
 <net name="SPW_SIN_N" class="0">
@@
 <wire x1="241.3" y1="129.54" x2="248.92" y2="129.54" width="0.1524" layer="91"/>
 </segment>
+<segment>
+<pinref part="J2" gate="G$1" pin="SIN-"/>
+<wire x1="287.02" y1="124.46" x2="284.48" y2="124.46" width="0.1524" layer="91"/>
+<label x="269.24" y="124.46" size="1.778" layer="95"/>
+</segment>
 </net>
 <net name="SPW_SIN_P" class="0">
@@
 <junction x="241.3" y="119.38"/>
 </segment>
+<segment>
+<pinref part="J2" gate="G$1" pin="SIN+"/>
+<wire x1="287.02" y1="127" x2="284.48" y2="127" width="0.1524" layer="91"/>
+<label x="269.24" y="127" size="1.778" layer="95"/>
+</segment>
 </net>
 <net name="SPW_DOUT_N" class="0">
@@
 <label x="238.76" y="109.22" size="1.778" layer="95"/>
 </segment>
+<segment>
+<pinref part="J2" gate="G$1" pin="DOUT-"/>
+<wire x1="287.02" y1="106.68" x2="284.48" y2="106.68" width="0.1524" layer="91"/>
+<label x="266.7" y="106.68" size="1.778" layer="95"/>
+</segment>
 </net>
 <net name="SPW_DOUT_P" class="0">
@@
 <label x="238.76" y="106.68" size="1.778" layer="95"/>
 </segment>
+<segment>
+<pinref part="J2" gate="G$1" pin="DOUT+"/>
+<wire x1="287.02" y1="109.22" x2="284.48" y2="109.22" width="0.1524" layer="91"/>
+<label x="266.7" y="109.22" size="1.778" layer="95"/>
+</segment>
 </net>
 <net name="SPW_SOUT_N" class="0">
@@
 <label x="238.76" y="104.14" size="1.778" layer="95"/>
 </segment>
+<segment>
+<pinref part="J2" gate="G$1" pin="SOUT-"/>
+<wire x1="287.02" y1="99.06" x2="284.48" y2="99.06" width="0.1524" layer="91"/>
+<label x="266.7" y="99.06" size="1.778" layer="95"/>
+</segment>
 </net>
 <net name="SPW_SOUT_P" class="0">
@@
 <label x="238.76" y="101.6" size="1.778" layer="95"/>
 </segment>
+<segment>
+<pinref part="J2" gate="G$1" pin="SOUT+"/>
+<wire x1="287.02" y1="101.6" x2="284.48" y2="101.6" width="0.1524" layer="91"/>
+<label x="266.7" y="101.6" size="1.778" layer="95"/>
+</segment>
 </net>
 <net name="N$64" class="0">
@@
 </segment>
 </net>
+<net name="N$93" class="0">
+<segment>
+<pinref part="J2" gate="G$1" pin="GND1"/>
+<wire x1="287.02" y1="116.84" x2="284.48" y2="116.84" width="0.1524" layer="91"/>
+</segment>
+</net>
 </nets>
 </sheet>
@@
 <instance part="R302" gate="R" x="73.66" y="5.08" rot="R180"/>
 <instance part="R303" gate="R" x="81.28" y="0" rot="R270"/>
-<instance part="U$23" gate="Q" x="109.22" y="20.32"/>
+<instance part="U303" gate="Q" x="109.22" y="20.32"/>
 <instance part="P+5" gate="1" x="111.76" y="33.02"/>
 </instances>
@@
 </segment>
 <segment>
-<pinref part="U$23" gate="Q" pin="D"/>
+<pinref part="U303" gate="Q" pin="D"/>
 <wire x1="111.76" y1="15.24" x2="111.76" y2="5.08" width="0.1524" layer="91"/>
 <wire x1="111.76" y1="5.08" x2="119.38" y2="5.08" width="0.1524" layer="91"/>
@@
 <wire x1="88.9" y1="20.32" x2="104.14" y2="20.32" width="0.1524" layer="91"/>
 <junction x="88.9" y="20.32"/>
-<pinref part="U$23" gate="Q" pin="G"/>
+<pinref part="U303" gate="Q" pin="G"/>
 </segment>
 </net>
@@
 </segment>
 <segment>
-<pinref part="U$23" gate="Q" pin="S"/>
+<pinref part="U303" gate="Q" pin="S"/>
 <pinref part="P+5" gate="1" pin="+12V"/>
 <wire x1="111.76" y1="30.48" x2="111.76" y2="25.4" width="0.1524" layer="91"/>

Commit message: first board layout completed
Parts:
- renumbered TP_PRE_IN1 to P_IN0, TP_PRE_IN2 to P_IN1, TP_PRE_IN3 to P_IN2, TP_PRE_IN4 to P_IN3, TP_PRE_OUT0 to P_OUT0, TP_PRE_OUT1 to P_OUT1, TP_PRE_OUT2 to P_OUT2, TP_PRE_OUT3 to P_OUT3, U1 to U111, U2 to U121, U3 to U131

Commit message: board layout completed, 100% routerd, logo inserted
Parts:
- added JP101: (no value), pinhead:PINHD-1X6
- added TP_GND, TP_GND1, TP_GND2: TPPAD1-13, Aardvark:TPPAD1-13
- added U$23, U$24, U$25, U$26: NC, Aardvark:NC
- J181: value (none) -> USB Mini-B Connector
- P_IN0, P_IN1, P_IN2, P_IN3, P_OUT0, P_OUT1, P_OUT2, P_OUT3, TP100, TP101, TP102, TP103, TP104, TP113, TP123, TP133, TP5, TP_1PPS, TP_2V5: value TPPAD1-17 -> TPPAD1-13; device Aardvark:TPPAD1-17 -> Aardvark:TPPAD1-13
- R190, R191, VR100, VR110, VR120, VR130: value (none) -> 1k
- R195, R196: value (none) -> 100
- U102, U112, U122, U132: value (none) -> LM6142
- U190: value (none) -> SN65LVDS049
- VR300, VR301: value (none) -> 5k
Connections:
- removed net AAA: J180.B_31
- removed net BBB: J180.A_2
- removed net N$34: J181.GND@1, J181.GND@2, J181.GND@3, J181.GND@4
- removed net N$93: J2.GND1
- removed net NNN: J180.A_6
- new net FPGA_GPIO0: J180.B_31, JP101.5
- new net FT232_/CTS_FPGA_/RTS: IC100.!CTS, J180.A_2
- new net FT232_/RTS_FPGA_/CTS: IC100.!RTS, J180.A_3
- new net TRIG_OUT0: J180.A_4, JP101.1
- new net TRIG_OUT1: J180.A_5, JP101.2
- new net TRIG_OUT2: J180.A_6, JP101.3
- new net TRIG_OUT3: J180.A_7, JP101.4
- net ADC2_D7: now also J180.A_15
- net GND: now also J181.GND@1, J181.GND@2, J181.GND@3, J181.GND@4, J2.GND1, JP101.6, TP_GND.TP, TP_GND1.TP, TP_GND2.TP
- net N$24: now also IC100.!DCD, U$23.NC; no longer J180.A_4
- net N$26: now also IC100.!DSR, U$24.NC; no longer J180.A_7
- net N$27: now also IC100.!DTR, U$25.NC; no longer J180.A_5
- net N$28: now also IC100.!RI, U$26.NC; no longer J180.A_3
Other:
- note removed: "TODO: Flow control signal between FPGA and FT232"
- moved on the sheet: JP100
