File: G_FY2015_Mez.sch (EAGLE design)
At the start: 197 parts, among them IC100 FT232RL, J1 RPI2_GPIO_HOLES, J100 EPL.00.250.NTN, J101 EPL.00.250.NTN, J102 EPL.00.250.NTN, J103 EPL.00.250.NTN, J180 TOKUDEN_SP6, J181 USB Mini-B Connector, J2 SPACEWIRE_MDMMDM9, J300 SHV_PIGTAIL_LAND, J301 SHV_PIGTAIL_LAND, J600_12V IL-4P-S3EN2, J610 2.1MMJACKTHM, U10 LM60, U100 AD9215, U101 AD8138, U102 LM6142, U11 MCP4822-E/SN, U110 AD9215, U111 AD8138, U112 LM6142, U120 AD9215, U121 AD8138, U122 LM6142, U130 AD9215, U131 AD8138, U132 LM6142, U190 SN65LVDS049, U191 GPS_FGPMMOPA6H, U192 LED-5, U300 OPTON_1PA_12, U301 OPTON_1PA_12, U302 2SC1815, U303 2SJ313, U5 MCP3208-CI/SL, U500 LT6106, U510 LT6106, U6 MCP1525TSOT-23-3, U600 PHT12050WAH, U610 PHT12050WAH, U620 LTC1983ES6-3, U7 LM60, U8 LM60, U9 LM60

Commit message: version 20150904 (placement completed; before replacing with complementray SMD resistor and cap)
Parts:
- removed C192: 100n, Aardvark:C226-3216
- removed C193: 4.7u, Aardvark:C226-3216
- removed J102, J103: EPL.00.250.NTN, Aardvark:EPL.00.250.NTN
- removed JP1: (no value), pinhead:PINHD-2X2
- removed JP100, TP_SPI: (no value), pinhead:PINHD-1X5
- removed JP101: (no value), pinhead:PINHD-1X6
- removed P_IN0, P_IN1, P_IN2, P_IN3, TP5: TPPAD1-13, Aardvark:TPPAD1-13
- removed R195, R196: 100, Aardvark:R2012
- removed SJ1: (no value), Aardvark:SJ2WW
- removed U10, U9: LM60, Aardvark:LM60
- removed U11: MCP4822-E/SN, Aardvark:MCP4822-E/SN
- removed U190: SN65LVDS049, Aardvark:SN65LVDS049
- added C18: 1u, Aardvark:C226-3216
- added C20, C22, C24, C26: 10u, Aardvark:C226-3216
- added C21, C23, C25: 0.1u, Aardvark:C226-3216
- added J110, J120, J130: EPL.00.250.NTN, Aardvark:EPL.00.250.NTN
- added J111, J121, J131, J620: IL-2P-S3EN2, Aardvark:IL-2P-S3EN2
- added J3: IL-3P-S3EN2, Aardvark:IL-3P-S3EN2
- added J4_I2C, J650_VOUT: IL-4P-S3EN2, Aardvark:IL-4P-S3EN2
- added J630, J640: USB_TYPEA_LUMBERG_2410_01, Aardvark:USB_TYPEA_LUMBERG_2410_01
- added JP101_TRIG_OUT: (no value), Aardvark:PINHD-2X7
- added JP_LCD: LCD16X2, Aardvark:LCD16X2
- added JP_SPI: (no value), Aardvark:PINHD-1X5
- added R109, R119, R129, R139: 50, Aardvark:R2012
- added R192: 2k, Aardvark:R2012
- added R193: 1k, Aardvark:R2012
- added SJ100, SJ110, SJ120, SJ130, SJ_ADC_MODE: (no value), Aardvark:SJ2WW
- added U$27, U$28, U$29, U$30, U$31, U$32, U$33, U$34, U$35, U$36, U$37, U$38, U$39, U$40: NC, Aardvark:NC
- added VR_CONT: (no value), Aardvark:DIP-TRIMMER-10K-10%-1/2W(3P-9.7X5.0X9.80MM)
- C19: value 100n -> 0.1u
- J101: value EPL.00.250.NTN -> IL-2P-S3EN2; device Aardvark:EPL.00.250.NTN -> Aardvark:IL-2P-S3EN2
- J2: value SPACEWIRE_MDMMDM9 -> IL-3P-S3EN2; device Aardvark:SPACEWIRE_MDMMDM9 -> Aardvark:IL-3P-S3EN2
- R190: value 1k -> 3k
- R500, R510: value 0.1 -> 0.01
- U100, U110, U120, U130: value AD9215 -> AD9215LONG_PAD; device Aardvark:AD9215 -> Aardvark:AD9215LONG_PAD
- VR100, VR110, VR120, VR130: value 1k -> (none)
Connections:
- removed net SLOWDAC_/LDAC: J1.GPIO2, U11A.!LDAC
- removed net SLOWDAC_0: JP1.1, U11A.V_OUTA
- removed net SLOWDAC_1: JP1.3, U11A.V_OUTB
- removed net SPW_DIN_N: J2.DIN-, R195.2, U190.RIN1-
- removed net SPW_DIN_P: J2.DIN+, R195.1, U190.RIN1+
- removed net SPW_DOUT_N: J2.DOUT-, U190.DOUT1-
- removed net SPW_DOUT_P: J2.DOUT+, U190.DOUT1+
- removed net SPW_SIN_N: J2.SIN-, R196.2, U190.RIN2-
- removed net SPW_SIN_P: J2.SIN+, R196.1, U190.RIN2+
- removed net SPW_SOUT_N: J2.SOUT-, U190.DOUT2-
- removed net SPW_SOUT_P: J2.SOUT+, U190.DOUT2+
- removed net VREF_3V3_1/2: R190.2, R191.1, SJ1.1
- new net LCD_D4: J1.GPIO6, JP_LCD.D4
- new net LCD_D5: J1.GPIO13, JP_LCD.D5
- new net LCD_D6: J1.GPIO19, JP_LCD.D6
- new net LCD_D7: J1.GPIO26, JP_LCD.D7
- new net LCD_ENA: J1.GPIO21, JP_LCD.ENABLE
- new net LCD_RS: J1.GPIO20, JP_LCD.RS
- new net LCD_V_CONT: JP_LCD.V_CONT, VR_CONT.2
- new net N$100: P_OUT0.TP, R109.2, U102B.OUT, VR100.2
- new net N$101: R109.1, SJ100.1
- new net N$102: R119.1, SJ110.1
- new net N$103: R129.1, SJ120.1
- new net N$104: R139.1, SJ130.1
- new net N$34: J630.DM, U$31.NC
- new net N$88: J630.DP, U$30.NC
- new net N$89: J640.DM, U$28.NC
- new net N$90: J640.DP, U$27.NC
- new net N$91: JP101_TRIG_OUT.11
- new net N$92: P_OUT1.TP, R119.2, U112B.OUT, VR110.2
- new net N$93: P_OUT2.TP, R129.2, U122B.OUT, VR120.2
- new net N$94: JP_LCD.D1, U$37.NC
- new net N$95: JP_LCD.D2, U$38.NC
- new net N$96: JP_LCD.D3, U$39.NC
- new net N$97: JP_LCD.D0, U$40.NC
- new net N$98: P_OUT3.TP, R139.2, U132B.OUT, VR130.2
- new net N$99: R192.2, R193.1, SJ_ADC_MODE.3
- new net RPI_I2C_SCL: J1.GPIO3, J4_I2C.2
- new net RPI_I2C_SDA: J1.GPIO2, J4_I2C.3
- net +3V3: now also C18.2, C20.2, C21.2, C22.2, C23.2, C24.2, C25.2, C26.2, J2.1, J3.1, J4_I2C.1, J650_VOUT.2, JP101_TRIG_OUT.14, R192.1; no longer C190.1, C191.1, C192.2, C193.2, IC100.VCC, IC100.VCCIO, U10.VDD, U11P.V_DD, U190.EN, U190.VCC, U9.VDD
- net +5V: now also C190.1, C191.1, IC100.VCC, IC100.VCCIO, J620.1, J630.VCC, J640.VCC, J650_VOUT.1, JP101_TRIG_OUT.2, JP_LCD.VCC, VR_CONT.1; no longer J180.V5
- net -3V3: now also J650_VOUT.3
- net ADC_CM: now also R190.2, R191.1; no longer SJ1.2
- net ADC_MODE: now also SJ_ADC_MODE.2; no longer J180.B_21
- net AGND: now also VR100.3, VR110.3, VR120.3, VR130.3; no longer VR100.1, VR110.1, VR120.1, VR130.1
- net FPGA_GPIO0: now also JP101_TRIG_OUT.9; no longer JP101.5
- net GND: now also C18.1, C20.1, C21.1, C22.1, C23.1, C24.1, C25.1, C26.1, J110.GND, J120.GND, J130.GND, J2.3, J3.3, J4_I2C.4, J620.2, J630.GND, J630.GND@1, J630.GND@2, J640.GND, J640.GND@1, J640.GND@2, J650_VOUT.4, JP101_TRIG_OUT.13, JP_LCD.GND, JP_LCD.R/W, R193.2, SJ_ADC_MODE.1, VR300.3, VR301.3, VR_CONT.3; no longer C192.1, C193.1, J101.GND, J102.GND, J103.GND, J180.GND, J2.GND, J2.GND1, J2.GND2, JP1.2, JP1.4, JP101.6, U10.GND, U11P.V_SS, U190.!EN, U190.GND, U9.GND, VR300.1, VR301.1
- net N$21: now also U$32.NC; no longer JP100.1
- net N$22: now also U$33.NC; no longer JP100.2
- net N$29: now also U$34.NC; no longer JP100.3
- net N$30: now also U$35.NC; no longer JP100.4
- net N$31: now also U$36.NC; no longer JP100.5
- net N$35: now also U$29.NC; no longer TP5.TP
- net N$5: now also VR300.1; no longer VR300.3
- net N$58: no longer P_IN0.TP
- net N$62: now also VR100.1; no longer VR100.2
- net N$7: now also VR301.1; no longer VR301.3
- net N$70: now also J110.1; no longer J101.1, P_IN1.TP
- net N$72: now also VR110.1; no longer VR110.2
- net N$75: now also J120.1; no longer J102.1, P_IN2.TP
- net N$77: now also VR120.1; no longer VR120.2
- net N$80: now also J130.1; no longer J103.1, P_IN3.TP
- net N$82: now also VR130.1; no longer VR130.2
- net PREAMP0_OUT: now also SJ100.2; no longer P_OUT0.TP, U102B.OUT, VR100.3
- net PREAMP1_OUT: now also SJ110.2; no longer P_OUT1.TP, U112B.OUT, VR110.3
- net PREAMP2_OUT: now also SJ120.2; no longer P_OUT2.TP, U122B.OUT, VR120.3
- net PREAMP3_OUT: now also SJ130.2; no longer P_OUT3.TP, U132B.OUT, VR130.3
- net SLOWADC_0: no longer SJ1.3
- net SLOWADC_2: now also J3.2; no longer U9.VOUT
- net SLOWADC_3: now also J2.2; no longer U10.VOUT
- net SPI_CE0: now also JP_SPI.4; no longer TP_SPI.4
- net SPI_CE1: now also JP_SPI.5; no longer TP_SPI.5, U11A.!CS
- net SPI_MISO: now also JP_SPI.2; no longer TP_SPI.2
- net SPI_MOSI: now also JP_SPI.3; no longer TP_SPI.3, U11A.SDI
- net SPI_SCLK: now also JP_SPI.1; no longer TP_SPI.1, U11A.SCK
- net SPW_DIN: no longer U190.ROUT1
- net SPW_DOUT: no longer U190.DIN1
- net SPW_SIN: no longer U190.ROUT2
- net SPW_SOUT: no longer U190.DIN2
- net TRIG_OUT0: now also JP101_TRIG_OUT.1; no longer JP101.1
- net TRIG_OUT1: now also JP101_TRIG_OUT.3; no longer JP101.2
- net TRIG_OUT2: now also JP101_TRIG_OUT.5; no longer JP101.3
- net TRIG_OUT3: now also JP101_TRIG_OUT.7; no longer JP101.4
Other:
- note added: "16x2 LCD"
- note added: "ADC Mode selection"
- note added: "For PMT temp monitor"
- note added: "LM60 sensors connected via cable"
- note added: "Power Connectors (input)"
- note added: "Power Connectors (output)"
- note added: "To outside pressure sensor (I2C)"
- note added: "オープンにするとADC内部でpull downされ、「Offset binary」＋「Duty-ratio stabilizer disabled」で動作。"
- note removed: "ADC Common ModeをSolderJumperで選択すること。"
- note removed: "Power Connectors"
- note removed: "Slow DAC"
- note removed: "SpaceWire LVDS Tx/Rx"
- moved on the sheet: C100, C101, C102, C103, C110, C111, C112, C113, C120, C121, C122, C123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

Commit message: as of 20150911 (4ch, FT232RL) before adding FT245 for higher data transfer rate
Parts:
- removed U192: LED-5, Aardvark:LED-5
- added C623, C624: 10u, Aardvark:C226-3216
- added C625: 1u, Aardvark:C226-3216
- added J_UART: IL-3P-S3EN2, Aardvark:IL-3P-S3EN2
- added LED_5V, LED_GPS, LED_HV: LED_1608, Aardvark:LED_1608
- added R304, R305: 1.2k, Aardvark:R2012
- added R601: 82, Aardvark:R2012
- added SJ101, SJ111, SJ121, SJ131: (no value), Aardvark:SJ2WW
- added U621: LTC1983ES6-5, Aardvark:LTC1983ES6-5
- C100, C110, C120, C130, C191: device Aardvark:C226-3216 -> Aardvark:C2012
- C190: value 100n -> 0.1u
- C194: device Aardvark:C226-3216 -> Aardvark:C1608
- R100, R105, R106, R110, R115, R116, R120, R125, R126, R130, R135, R136: value 49.9 -> 51
- R101, R103, R104, R111, R113, R114, R121, R123, R124, R131, R133, R134: value 499 -> 510
- R102, R112, R122, R132: value 523 -> 510
- R109, R119, R129, R139: value 50 -> 51
- R199: value 330 -> 82
- R600: value 280 -> 270
- R610: device Aardvark:R2012 -> Aardvark:R1608
- U102, U112, U122, U132: value LM6142 -> LM6172
Connections:
- new net -5V: C103.2, C113.2, C123.2, C133.2, C624.1, U102P.V-, U112P.V-, U122P.V-, U132P.V-, U621.VOUT
- new net AIN_0: J100.1, J101.1, SJ100.3, SJ101.1
- new net AIN_1: C110.1, R117.2, SJ110.3, SJ111.2, U112A.-
- new net AIN_2: J120.1, J121.1, SJ120.3, SJ121.1
- new net AIN_3: J130.1, J131.1, SJ130.3, SJ131.1
- new net N$105: J110.1, J111.1, SJ111.1
- new net N$106: C100.1, R107.2, SJ101.2, U102A.-
- new net N$108: C625.2, U621.C+
- net +3V3: no longer C102.2, C112.2, C122.2, C132.2, U102P.V+, U112P.V+, U122P.V+, U132P.V+
- net +5V: now also C102.2, C112.2, C122.2, C132.2, C623.2, R601.2, U102P.V+, U112P.V+, U122P.V+, U132P.V+, U621./SHDN, U621.VCC
- net -3V3: no longer C103.2, C113.2, C123.2, C133.2, U102P.V-, U112P.V-, U122P.V-, U132P.V-
- net GND: now also C623.1, C624.2, J101.2, J111.2, J121.2, J131.2, J_UART.3, LED_5V.C, LED_GPS.C, LED_HV.C, R101.1, R111.1, R121.1, R131.1, U621.GND; no longer R102.2, R112.2, R122.2, R132.2, U192.K
- net HV_PWR_12V: now also R304.2, R305.2
- net N$58: now also LED_HV.A, R304.1, R305.1; no longer C100.1, J100.1, R107.2, U102A.-
- net N$69: now also LED_GPS.A; no longer U192.A
- net N$70: now also LED_5V.A, R601.1; no longer C110.1, J110.1, R117.2, U112A.-
- net N$75: now also C130.1, R137.2, SJ131.2, U132A.-; no longer C120.1, J120.1, R127.2, U122A.-
- net N$80: now also C120.1, R127.2, SJ121.2, U122A.-; no longer C130.1, J130.1, R137.2, U132A.-
- net N$91: now also C625.1, U621.C-; no longer JP101_TRIG_OUT.11
- net PREAMP0_OUT: now also R102.2; no longer R101.1
- net PREAMP1_OUT: now also R112.2; no longer R111.1
- net PREAMP2_OUT: now also R122.2; no longer R121.1
- net PREAMP3_OUT: now also R132.2; no longer R131.1
- net RPI_RX_FPGA_TX: now also J_UART.1
- net RPI_TX_FPGA_RX: now also J_UART.2
Other:
- note added: "DCDC +5V=>--5V"
- note added: "Vf=1.9VでI=18mAの予定。"
- note added: "Vf=1.9Vで、LEDに18mA流れる予定。"
- note added: "パイロットランプ(5V)"
- note added: "合成抵抗600オーム。"
- note added: "本当はR100, R105, R106=49.9オーム"
- note added: "本当はR101=523オーム"
- note added: "本当はR102, R103, R104=499オーム"
- note added: "本当はR600=280オーム"
- moved on the sheet: J101, J111, J121, J131, TP100

Commit message: version B completed. before autoroute for P-ban submit
Parts:
- removed C1, C11, C12, C122, C123, C13, C132, C133, C15, C16, C19, C21, C23, C25, C3, C4, C5, C7, C8, C9: 0.1u, Aardvark:C226-3216
- removed C10, C14, C2, C20, C22, C24, C26, C6: 10u, Aardvark:C226-3216
- removed C120, C130: 100p, Aardvark:C2012
- removed C121, C131: ???, Aardvark:C226-3216
- removed JP101_TRIG_OUT: (no value), Aardvark:PINHD-2X7
- removed JP2: (no value), pinhead:PINHD-2X2
- removed LED_GPS: LED_1608, Aardvark:LED_1608
- removed P_OUT2, P_OUT3, TP100, TP104: TPPAD1-13, Aardvark:TPPAD1-13
- removed R127, R137: 1M, Aardvark:R2012
- removed R128, R138: ???, Aardvark:R2012
- removed R129, R139: 51, Aardvark:R2012
- removed R199: 82, Aardvark:R2012
- removed R304, R305: 1.2k, Aardvark:R2012
- removed SJ120, SJ121, SJ130, SJ131: (no value), Aardvark:SJ2WW
- removed U122, U132: LM6172, Aardvark:LM6172SOIC(D)8
- removed VR120, VR130: (no value), Aardvark:DIP-TRIMMER-10K-10%-1/2W(3P-9.7X5.0X9.80MM)
- added -3V, -5V, AIN1+, AIN1-, GPIO0, GPIO1, VR100PIN2, VR110PIN2, VR_HV0, VR_HV1: TPPAD1-13, Aardvark:TPPAD1-13
- added C104, C106, C107, C108, C114, C116, C117, C118, C124, C126, C127, C128, C134, C136, C137, C138, C192, C193: 0.1u, Aardvark:C2012
- added C105, C109, C115, C119, C125, C129, C135, C139: 10u, Aardvark:C2012
- added C197: 0.01u, Aardvark:C1608
- added C198: 10u, Aardvark:C226-3216
- added IC101: FT245RL, Aardvark:FT245RL
- added J182: USB Mini-B Connector, Aardvark:MINI-USB-RCPT-B-5PS-R/A-SMD(ST-USB-002A)
- added JP_ADC: (no value), Aardvark:PINHD-2X2
- added LED_5V_SW, LED_RPI: SML-311WTT86, Aardvark:LED_1608
- added R400: 680, Aardvark:R2012
- added R520: 47k, Aardvark:R2012
- added R521, R522: 4.7k, Aardvark:R2012
- added R523: 1.5k, Aardvark:R2012
- added R_PZC0, R_PZC1: 56k, Aardvark:R2012
- added U$13, U$14, U$15, U$16, U$41, U$42, U$43, U$44: NC, Aardvark:NC
- added U520: 2SC1815, Aardvark:2SC1815
- added U521: 2SJ681, Aardvark:2SJ681
- C101, C111: value ??? -> 200p; device Aardvark:C226-3216 -> Aardvark:C2012
- C102, C103, C112, C113: value 0.1u -> 0.033u; device Aardvark:C226-3216 -> Aardvark:C2012
- C190: device Aardvark:C226-3216 -> Aardvark:C2012
- C194: value 0.01u -> 4.7u; device Aardvark:C1608 -> Aardvark:C2012
- C195: value 10u -> 0.1u; device Aardvark:C226-3216 -> Aardvark:C2012
- LED_5V, LED_HV: value LED_1608 -> SML-311WTT86
- R107, R117: value 1M -> 100k
- R108, R118: value ??? -> 10k
- R301: value 47k -> 4.7k
- R601: value 82 -> 1.5k
- R610: device Aardvark:R1608 -> Aardvark:R2012
- U303: value 2SJ313 -> 2SJ681; device Aardvark:2SJ313 -> Aardvark:2SJ681
- VR100, VR110, VR_CONT: value (none) -> 5k
- renumbered C17 to C411, C18 to C410, J1 to J400, J2 to J411, J3 to J410, J4_I2C to J_I2C, TP101 to AIN0+, TP102 to AIN0-, TP103 to VREF0, TP113 to VREF1, TP123 to VREF2, TP133 to VREF3, TP_1PPS to 1PPS, TP_2V5 to 2.5V, TP_GND1 to GND, U5 to U410, U6 to U411, U7 to U412, U8 to U413
Connections:
- removed net AGND: VR100.3, VR110.3, VR120.3, VR130.3
- removed net FT232_/CTS_FPGA_/RTS: IC100.!CTS, J180.A_2
- removed net FT232_/RTS_FPGA_/CTS: IC100.!RTS, J180.A_3
- removed net N$103: R129.1, SJ120.1
- removed net N$104: R139.1, SJ130.1
- removed net N$77: U122B.-, VR120.1
- removed net N$78: C130.2, C131.1, R137.1, U132A.OUT
- removed net N$79: C131.2, R138.1, U132B.+
- removed net N$80: C120.1, R127.2, SJ121.2, U122A.-
- removed net N$82: U132B.-, VR130.1
- removed net N$86: R301.1, U302.C
- removed net N$93: P_OUT2.TP, R129.2, U122B.OUT, VR120.2
- removed net N$98: P_OUT3.TP, R139.2, U132B.OUT, VR130.2
- removed net PREAMP2_OUT: R120.2, R122.2, SJ120.2
- removed net PREAMP3_OUT: R130.2, R132.2, SJ130.2
- removed net RPI_RX_FPGA_TX: J180.B_22, J400.GPIO15, J_UART.1
- removed net RPI_TX_FPGA_RX: J180.B_24, J400.GPIO14, J_UART.2
- removed net SPW_DIN: J180.B_30
- removed net SPW_DOUT: J180.B_26
- removed net SPW_SIN: J180.B_32
- removed net SPW_SOUT: J180.B_28
- removed net TRIG_OUT0: J180.A_4, JP101_TRIG_OUT.1
- removed net TRIG_OUT1: J180.A_5, JP101_TRIG_OUT.3
- removed net TRIG_OUT2: J180.A_6, JP101_TRIG_OUT.5
- removed net TRIG_OUT3: J180.A_7, JP101_TRIG_OUT.7
- new net 5V_PWR_ENADIS: J400.GPIO12, R521.2
- new net 5V_SW_OUT: J630.VCC, R523.2, U521.D
- new net FPGA_GPIO1: GPIO1.TP, J180.A_7
- new net FT245_/RE: IC101._RD, J180.A_3
- new net FT245_/RXF: IC101._RXF, J180.B_21
- new net FT245_/TXE: IC101._TXE, J180.B_20
- new net FT245_D0: IC101.D0, J180.B_22
- new net FT245_D1: IC101.D1, J180.B_24
- new net FT245_D2: IC101.D2, J180.B_26
- new net FT245_D3: IC101.D3, J180.B_28
- new net FT245_D4: IC101.D4, J180.B_30
- new net FT245_D5: IC101.D5, J180.B_32
- new net FT245_D6: IC101.D6, J180.A_4
- new net FT245_D7: IC101.D7, J180.A_5
- new net FT245_WE: IC101.WR, J180.A_2
- new net N$107: IC101._RESET, U$13.NC
- new net N$109: IC101.OSCI, U$14.NC
- new net N$110: IC101.OSCO, U$15.NC
- new net N$111: IC101.3V3OUT, U$16.NC
- new net N$112: IC100.!RTS, U$43.NC
- new net N$113: IC100.!CTS, U$44.NC
- new net N$116: IC101.PWEN, U$41.NC
- new net RPI_LED0: J400.GPIO5, R400.2
- new net RPI_OUT_FPGA_IN0: J180.B_31, J400.GPIO4
- new net RPI_RX: J400.GPIO15, J_UART.1
- new net RPI_TX: J400.GPIO14, J_UART.2
- new net USB_D_M2: IC101.USBDM, J182.DM
- new net USB_D_P2: IC101.USBDP, J182.DP
- net +3V3: now also C108.2, C109.2, C118.2, C119.2, C128.2, C129.2, C138.2, C139.2, C192.1, C195.1, C197.2, C198.2, IC100.VCCIO, IC101.VCCIO; no longer C19.2, C194.2, C195.2, C20.2, C21.2, C22.2, C23.2, C24.2, C25.2, C26.2, JP101_TRIG_OUT.14
- net +5V: now also C193.1, C194.1, IC101.VCC, R520.2, U521.S; no longer C122.2, C132.2, IC100.VCCIO, J630.VCC, JP101_TRIG_OUT.2, U122P.V+, U132P.V+
- net -3V3: now also -3V.TP; no longer J650_VOUT.3
- net -5V: now also -5V.TP, J650_VOUT.3; no longer C123.2, C133.2, U122P.V-, U132P.V-
- net ADC0_CLK: no longer TP104.TP
- net ADC1_VIN_N: now also AIN1-.TP
- net ADC1_VIN_P: now also AIN1+.TP
- net ADC_PDWN: no longer J180.B_20
- net AIN_1: now also J110.1, J111.1, SJ111.1; no longer C110.1, R117.2, SJ111.2, U112A.-
- net AIN_2: now also R120.2, R122.2; no longer SJ120.3, SJ121.1
- net AIN_3: now also R130.2, R132.2; no longer SJ130.3, SJ131.1
- net FPGA_GPIO0: now also GPIO0.TP, J180.A_6; no longer J180.B_31, JP101_TRIG_OUT.9
- net GND: now also C106.2, C107.2, C108.1, C109.1, C116.2, C117.2, C118.1, C119.1, C126.2, C127.2, C128.1, C129.1, C136.2, C137.2, C138.1, C139.1, C192.2, C193.2, C194.2, C195.2, C197.1, C198.1, IC101.AGND, IC101.GND1, IC101.GND2, IC101.GND3, IC101.TEST, J182.GND@1, J182.GND@2, J182.GND@3, J182.GND@4, J182.GND@5, JP_ADC.2, JP_ADC.4, LED_5V_SW.C, LED_RPI.C, R302.2, R522.2, U520.E, VR100.1, VR110.1, VR300.1, VR301.1; no longer C11.2, C12.2, C122.1, C123.1, C132.1, C133.1, C15.2, C16.2, C19.1, C194.1, C195.1, C20.1, C21.1, C22.1, C23.1, C24.1, C25.1, C26.1, C3.2, C4.2, C7.2, C8.2, JP101_TRIG_OUT.13, JP2.2, JP2.4, LED_GPS.C, R128.2, R138.2, R303.2, U122A.+, U132A.+, VR300.3, VR301.3
- net HV_PWR_12V: now also R303.2; no longer R304.2, R305.2
- net HV_PWR_ENADIS: now also R301.2; no longer R302.2
- net N$100: now also VR100.3; no longer P_OUT0.TP, VR100.2
- net N$105: now also C110.1, R117.2, SJ111.2, U112A.-; no longer J110.1, J111.1, SJ111.1
- net N$11: now also C104.2, C105.2, C106.1; no longer C1.2, C2.2, C3.1
- net N$13: now also C114.2, C115.2, C116.1; no longer C5.2, C6.2, C7.1
- net N$14: now also C104.1, C105.1, C107.1; no longer C1.1, C2.1, C4.1
- net N$15: now also C114.1, C115.1, C117.1; no longer C5.1, C6.1, C8.1
- net N$17: now also C124.2, C125.2, C126.1; no longer C10.2, C11.1, C9.2
- net N$18: now also C124.1, C125.1, C127.1; no longer C10.1, C12.1, C9.1
- net N$20: now also C134.2, C135.2, C136.1; no longer C13.2, C14.2, C15.1
- net N$23: now also C134.1, C135.1, C137.1; no longer C13.1, C14.1, C16.1
- net N$3: now also VR_HV0.TP
- net N$5: now also VR300.3; no longer VR300.1
- net N$54: now also R_PZC0.1
- net N$55: now also R_PZC0.2
- net N$58: now also R303.1; no longer R304.1, R305.1
- net N$6: now also VR_HV1.TP
- net N$61: now also R_PZC1.1
- net N$62: now also U112B.-, VR110.2, VR110PIN2.TP; no longer U102B.-, VR100.1
- net N$63: now also R_PZC1.2
- net N$65: now also U$42.NC; no longer R199.2
- net N$69: now also LED_RPI.A, R400.1; no longer LED_GPS.A, R199.1
- net N$7: now also VR301.3; no longer VR301.1
- net N$72: now also R520.1, U520.C, U521.G; no longer U112B.-, VR110.1
- net N$73: now also U102B.-, VR100.2, VR100PIN2.TP; no longer C120.2, C121.1, R127.1, U122A.OUT
- net N$74: now also R521.1, R522.1, U520.B; no longer C121.2, R128.1, U122B.+
- net N$75: now also LED_5V_SW.A, R523.1; no longer C130.1, R137.2, SJ131.2, U132A.-
- net N$85: now also U302.C; no longer R301.2
- net N$87: now also R301.1; no longer R303.1
- net N$92: now also VR110.3; no longer P_OUT1.TP, VR110.2
- net PREAMP0_OUT: now also P_OUT0.TP; no longer TP100.TP
- net PREAMP1_OUT: now also P_OUT1.TP
- net SLOWADC_6: now also JP_ADC.1; no longer JP2.1
- net SLOWADC_7: now also JP_ADC.3; no longer JP2.3
Other:
- note added: "5V On/Off from Raspberry Pi"
- note added: "SENSEピンをGNDに落としているので、 differential spanは2V (±1V)で、Vref=1Vとなる。"
- note added: "Vf=1.8V / I_F=2mA"
- note added: "Vf=1.8V I_F=2mA"
- note removed: "Vf=1.9VでI=18mAの予定。"
- note removed: "Vf=1.9Vで、LEDに18mA流れる予定。"
- note removed: "合成抵抗600オーム。"
